Commit message: Attach tray to the URDF.

File: assets/combined.urdf (robot description, URDF)
Before this commit: robot ur5e, 13 links, 12 joints
Links:
- added link tray, mass 0.1; collision cylinder length=0.02 radius=0.15; visual cylinder length=0.02 radius=0.15
- link base_link_inertia: geometry collision mesh filename=file://meshes/base.stl; visual mesh filename=file://meshes/base.dae
- link forearm_link: geometry collision mesh filename=file://meshes/forearm.stl; visual mesh filename=file://meshes/forearm.dae
- link shoulder_link: geometry collision mesh filename=file://meshes/shoulder.stl; visual mesh filename=file://meshes/shoulder.dae
- link upper_arm_link: geometry collision mesh filename=file://meshes/upperarm.stl; visual mesh filename=file://meshes/upperarm.dae
- link wrist_1_link: geometry collision mesh filename=file://meshes/wrist1.stl; visual mesh filename=file://meshes/wrist1.dae
- link wrist_2_link: geometry collision mesh filename=file://meshes/wrist2.stl; visual mesh filename=file://meshes/wrist2.dae
- link wrist_3_link: geometry collision mesh filename=file://meshes/wrist3.stl; visual mesh filename=file://meshes/wrist3.dae
Joints:
- added joint tool_tray_joint: type fixed, parent tool0, child tray, origin xyz=0.0 0.0 0.25 rpy=1.5707963267948966 0 0

Commit message: Add basic simulation infrastructure.

File: assets/combined.urdf (robot description, URDF)
Before this commit: robot ur5e, 14 links, 13 joints
Joints:
- joint tool_tray_joint: origin xyz=0.0 0.0 0.25 rpy=1.5707963267948966 0 0 -> xyz=0.0 0.0 0.25 rpy=0 -1.5707963267948966 -1.5707963267948966

Commit message: Add more comments and extra touches.

File: assets/combined.urdf (robot description, URDF)
Before this commit: robot ur5e, 14 links, 13 joints
Joints:
- joint base_joint: origin xyz=0 0 0 rpy=0 0 0 -> xyz=0 0 1 rpy=0 0 0
